Commit message: 添加激光传感器和IMU链接及关节，更新URDF模型以支持新组件

File: demo_diff_robot/urdf/diff_robot.urdf.xacro (robot description, xacro)
@@ -10,4 +10,7 @@
     <xacro:property name="base_width" value="0.1"/>
     <xacro:property name="base_height" value="0.05"/>
+    <xacro:property name="laser_mass" value="0.03"/>
+    <xacro:property name="laser_length" value="0.01"/>
+    <xacro:property name="laser_radius" value="0.01"/>
     <xacro:property name="wheel_mass" value="0.3"/>
     <xacro:property name="wheel_length" value="0.020"/>
@@ -18,4 +21,5 @@
     <link name="${prefix}dummy_link">
     </link>
+    <!-- dummy joint -->
     <joint name="${prefix}dummy_joint" type="fixed">
       <parent link="${prefix}dummy_link"/>
@@ -43,4 +47,87 @@
       <material>Gazebo/Orange</material>
     </gazebo>
+    <!-- imu link -->
+    <link name="${prefix}imu_link">
+      <visual>
+        <origin xyz="0 0 0" rpy="0 0 0"/>
+        <geometry>
+          <box size="0.01 0.01 0.01"/>
+        </geometry>
+        <material name="red"/>
+      </visual>
+      <collision>
+        <origin xyz="0 0 0" rpy="0 0 0"/>
+        <geometry>
+          <box size="0.01 0.01 0.01"/>
+        </geometry>
+      </collision>
+      <xacro:box_inertia m="0.01" l="0.01" w="0.01" h="0.01"/>
+    </link>
+    <!-- imu joint -->
+    <joint name="${prefix}imu_joint" type="fixed">
+      <parent link="${prefix}base_link"/>
+      <child link="${prefix}imu_link"/>
+      <origin xyz="0 0 0" rpy="0 0 0"/>
+    </joint>
+    <!-- laser link -->
+    <link name="${prefix}laser_link">
+      <visual>
+        <origin xyz="0 0 0" rpy="0 0 0"/>
+        <geometry>
+          <cylinder length="${laser_length}" radius="${laser_radius}"/>
+        </geometry>
+        <material name="red"/>
+      </visual>
+      <collision>
+        <origin xyz="0 0 0" rpy="0 0 0"/>
+        <geometry>
+          <cylinder length="${laser_length}" radius="${laser_radius}"/>
+        </geometry>
+      </collision>
+      <xacro:cylinder_inertia m="${laser_mass}" l="${laser_length}" r="${laser_radius}"/>
+    </link>
+    <gazebo reference="${prefix}laser_link">
+      <material>Gazebo/Red</material>
+      <sensor name="laser_scan" type="ray">
+        <plugin name="laser_scan" filename="libgazebo_ros_ray_sensor.so">
+          <ros>
+            <namespace>/</namespace>
+            <remapping>~/out:=/scan</remapping>
+          </ros>
+          <output_type>sensor_msgs/LaserScan</output_type>
+          <frame_name>laser_link</frame_name>
+        </plugin>
+        <always_on>true</always_on>
+        <visualize>true</visualize>
+        <update_rate>10</update_rate>
+        <pose>0 0 0 0 0 0</pose>
+        <ray>
+          <scan>
+            <horizontal>
+              <samples>360</samples>
+              <resolution>1</resolution>
+              <min_angle>-${PI}</min_angle>
+              <max_angle>${PI}</max_angle>
+            </horizontal>
+          </scan>
+          <range>
+            <min>0.03</min>
+            <max>5</max>
+            <resolution>0.003</resolution>
+          </range>
+          <noise>
+            <type>gaussian</type>
+            <mean>0.0</mean>
+            <stddev>0.01</stddev>
+          </noise>
+        </ray>
+      </sensor>
+    </gazebo>
+    <!-- laser joint -->
+    <joint name="${prefix}laser_joint" type="fixed">
+      <parent link="${prefix}base_link"/>
+      <child link="${prefix}laser_link"/>
+      <origin xyz="0 0 ${base_height/2 + laser_length/2}" rpy="0 0 0"/>
+    </joint>
     <!-- left wheel link -->
     <link name="${prefix}left_wheel_link">

Commit message: 将激光传感器更名为激光雷达，更新相关属性和传感器配置

File: demo_diff_robot/urdf/diff_robot.urdf.xacro (robot description, xacro)
@@ -10,7 +10,7 @@
     <xacro:property name="base_width" value="0.1"/>
     <xacro:property name="base_height" value="0.05"/>
-    <xacro:property name="laser_mass" value="0.03"/>
-    <xacro:property name="laser_length" value="0.01"/>
-    <xacro:property name="laser_radius" value="0.01"/>
+    <xacro:property name="lidar_mass" value="0.03"/>
+    <xacro:property name="lidar_length" value="0.01"/>
+    <xacro:property name="lidar_radius" value="0.01"/>
     <xacro:property name="wheel_mass" value="0.3"/>
     <xacro:property name="wheel_length" value="0.020"/>
@@ -64,4 +64,21 @@
       <xacro:box_inertia m="0.01" l="0.01" w="0.01" h="0.01"/>
     </link>
+    <gazebo reference="${prefix}imu_link">
+      <material>Gazebo/Red</material>
+      <sensor name="imu_sensor" type="imu">
+        <plugin name="imu_sensor" filename="libgazebo_ros_imu.so">
+          <ros>
+            <namespace>/</namespace>
+            <remapping>~/out:=/imu</remapping>
+          </ros>
+          <output_type>sensor_msgs/Imu</output_type>
+          <frame_name>imu_link</frame_name>
+        </plugin>
+        <always_on>true</always_on>
+        <visualize>true</visualize>
+        <update_rate>10</update_rate>
+        <pose>0 0 0 0 0 0</pose>
+      </sensor>
+    </gazebo>
     <!-- imu joint -->
     <joint name="${prefix}imu_joint" type="fixed">
@@ -70,10 +87,10 @@
       <origin xyz="0 0 0" rpy="0 0 0"/>
     </joint>
-    <!-- laser link -->
-    <link name="${prefix}laser_link">
-      <visual>
-        <origin xyz="0 0 0" rpy="0 0 0"/>
-        <geometry>
-          <cylinder length="${laser_length}" radius="${laser_radius}"/>
+    <!-- lidar link -->
+    <link name="${prefix}lidar_link">
+      <visual>
+        <origin xyz="0 0 0" rpy="0 0 0"/>
+        <geometry>
+          <cylinder length="${lidar_length}" radius="${lidar_radius}"/>
         </geometry>
         <material name="red"/>
@@ -82,13 +99,13 @@
         <origin xyz="0 0 0" rpy="0 0 0"/>
         <geometry>
-          <cylinder length="${laser_length}" radius="${laser_radius}"/>
-        </geometry>
-      </collision>
-      <xacro:cylinder_inertia m="${laser_mass}" l="${laser_length}" r="${laser_radius}"/>
-    </link>
-    <gazebo reference="${prefix}laser_link">
+          <cylinder length="${lidar_length}" radius="${lidar_radius}"/>
+        </geometry>
+      </collision>
+      <xacro:cylinder_inertia m="${lidar_mass}" l="${lidar_length}" r="${lidar_radius}"/>
+    </link>
+    <gazebo reference="${prefix}lidar_link">
       <material>Gazebo/Red</material>
-      <sensor name="laser_scan" type="ray">
-        <plugin name="laser_scan" filename="libgazebo_ros_ray_sensor.so">
+      <sensor name="lidar_sensor" type="ray">
+        <plugin name="lidar_sensor" filename="libgazebo_ros_ray_sensor.so">
           <ros>
             <namespace>/</namespace>
@@ -96,5 +113,5 @@
           </ros>
           <output_type>sensor_msgs/LaserScan</output_type>
-          <frame_name>laser_link</frame_name>
+          <frame_name>lidar_link</frame_name>
         </plugin>
         <always_on>true</always_on>
@@ -124,9 +141,9 @@
       </sensor>
     </gazebo>
-    <!-- laser joint -->
-    <joint name="${prefix}laser_joint" type="fixed">
-      <parent link="${prefix}base_link"/>
-      <child link="${prefix}laser_link"/>
-      <origin xyz="0 0 ${base_height/2 + laser_length/2}" rpy="0 0 0"/>
+    <!-- lidar joint -->
+    <joint name="${prefix}lidar_joint" type="fixed">
+      <parent link="${prefix}base_link"/>
+      <child link="${prefix}lidar_link"/>
+      <origin xyz="0 0 ${base_height/2 + lidar_length/2}" rpy="0 0 0"/>
     </joint>
     <!-- left wheel link -->

Commit message: 更新差分机器人配置，修正基础框架链接和关节名称，优化 RViz 可视化设置

File: demo_diff_robot/urdf/diff_robot.urdf.xacro (robot description, xacro)
@@ -18,10 +18,10 @@
     <xacro:property name="caster_wheel_mass" value="0.1"/>
     <xacro:property name="caster_wheel_radius" value="0.015"/>
-    <!-- dummy link -->
-    <link name="${prefix}dummy_link">
-    </link>
-    <!-- dummy joint -->
-    <joint name="${prefix}dummy_joint" type="fixed">
-      <parent link="${prefix}dummy_link"/>
+    <!-- base footprint link -->
+    <link name="${prefix}base_footprint">
+    </link>
+    <!-- base footprint joint -->
+    <joint name="${prefix}base_footprint_joint" type="fixed">
+      <parent link="${prefix}base_footprint"/>
       <child link="${prefix}base_link"/>
       <origin xyz="0 0 ${base_height/2+wheel_radius}" rpy="0 0 0"/>
